File: electronics/RAMPlatterHybrid.kicad_pcb (KiCad board)
At the start: 2 copper layers, 65 x 56 mm, 39 parts, among them J1 Raspberry_Pi_2_3, U1 LM358, U2 74LVC74APW, U3 AV2-8.4-10, U4 AV2-8.4-10, U5 HC4046A, U6 CD74HC4059, U7 AP1117-33, U8 WM8750

Commit message: v1.0
Parts:
- added C10: 10u, Capacitor_SMD:CP_Elec_4x5.3, F.Cu at (231.5, 111.5)
- added C11: 1u NP, Capacitor_SMD:CP_Elec_5x5.3, F.Cu at (240.5, 129.5)
- added C12: 1u NP, Capacitor_SMD:CP_Elec_5x5.3, F.Cu at (240.5, 135.3)
- added C13: 1u NP, Capacitor_SMD:CP_Elec_5x5.3, F.Cu at (216.2, 131.2)
- added C14: 1u NP, Capacitor_SMD:CP_Elec_5x5.3, F.Cu at (210.4, 131.2)
- added C16: 10u, Capacitor_SMD:CP_Elec_4x5.3, F.Cu at (234.0, 126.8)
- added C8: 10u, Capacitor_SMD:CP_Elec_4x5.3, F.Cu at (223.6, 129.6)
- added J2: Raspberry_Pi_2_3, Connector_PinHeader_2.54mm:PinHeader_2x20_P2.54mm_Vertical, F.Cu at (208.8, 89.0)
- added JP3: SolderJumper_2_Bridged, Jumper:SolderJumper-2_P1.3mm_Bridged_Pad1.0x1.5mm, B.Cu at (229.2, 120.0)
- J1: footprint Connector_PinHeader_2.54mm:PinHeader_2x20_P2.54mm_Vertical -> 40pin.SMD.rev:02x20.SMD.pinLocsRev; moved to B.Cu
- R10, R7, R8, R9: value 47R -> 75R
- moved R12 55.3 mm to (244.2, 121.5)
- moved C23 55.1 mm to (233.5, 121.5)
- moved R11 55.1 mm to (239.2, 125.0)
- moved U5 55.1 mm to (238.3, 119.0)
- moved JP2 55.0 mm to (261.2, 110.7), turned to 90 degrees
- moved C20 53.6 mm to (242.2, 125.0)
- moved R6 53.5 mm to (210.5, 136.8), turned to 90 degrees
- moved C21 53.2 mm to (240.4, 112.2), turned to 90 degrees
- moved JP1 51.7 mm to (242.4, 111.2), turned to 90 degrees
- moved U6 48.1 mm to (251.7, 107.3), turned to 90 degrees
- moved R5 45.1 mm to (216.2, 136.8), turned to 90 degrees
- moved C17 44.3 mm to (228.0, 126.5), turned to 270 degrees
- moved R10 40.2 mm to (227.5, 116.9), turned to 90 degrees
- moved C22 39.3 mm to (242.5, 102.2), turned to 180 degrees
- moved C15 38.4 mm to (229.5, 126.5), turned to 270 degrees
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Connections:
- net Net-(C4-Pad1) renamed /AVDD
- J1 pad 1: +3V3 -> Net-(J1-Pad1)
- J1 pad 10: (no net) -> Net-(J1-Pad10)
- J1 pad 11: (no net) -> Net-(J1-Pad11)
- J1 pad 13: (no net) -> Net-(J1-Pad13)
- J1 pad 15: (no net) -> Net-(J1-Pad15)
- J1 pad 16: (no net) -> Net-(J1-Pad16)
- J1 pad 18: (no net) -> Net-(J1-Pad18)
- J1 pad 19: (no net) -> Net-(J1-Pad19)
- J1 pad 21: (no net) -> Net-(J1-Pad21)
- J1 pad 22: (no net) -> Net-(J1-Pad22)
- J1 pad 23: (no net) -> Net-(J1-Pad23)
- J1 pad 24: (no net) -> Net-(J1-Pad24)
- J1 pad 26: (no net) -> Net-(J1-Pad26)
- J1 pad 27: (no net) -> Net-(J1-Pad27)
- J1 pad 28: (no net) -> Net-(J1-Pad28)
- J1 pad 29: (no net) -> Net-(J1-Pad29)
- J1 pad 31: (no net) -> Net-(J1-Pad31)
- J1 pad 32: (no net) -> Net-(J1-Pad32)
- J1 pad 33: (no net) -> Net-(J1-Pad33)
- J1 pad 36: (no net) -> Net-(J1-Pad36)
- J1 pad 7: (no net) -> Net-(J1-Pad7)
- J1 pad 8: (no net) -> Net-(J1-Pad8)
- R5 pad 2: (no net) -> Net-(C13-Pad2)
- R6 pad 2: (no net) -> Net-(C14-Pad2)
- U6 pad 14: /LOW -> /HIGH
- U8 pad 12: (no net) -> Net-(C14-Pad1)
- U8 pad 13: (no net) -> Net-(C13-Pad1)
- U8 pad 27: (no net) -> Net-(C12-Pad1)
- U8 pad 28: (no net) -> Net-(C11-Pad1)
Routing:
- net +3V3: track 0.00 -> 128.5 mm, vias 0 -> 6
- net +5V: track 0.00 -> 58.2 mm, vias 0 -> 2
- net /HIGH: track 0.00 -> 54.9 mm, vias 0 -> 11
- net /LOW: track 0.00 -> 52.9 mm, vias 0 -> 11
- net /SDA: track 0.00 -> 51.2 mm, vias 0 -> 1
- net /SCL: track 0.00 -> 49.7 mm, vias 0 -> 1
- net Net-(R8-Pad1): track 0.00 -> 44.8 mm
- net /I2S_ADC: track 0.00 -> 44.2 mm, vias 0 -> 1
- net /Rin: track 0.00 -> 41.5 mm
- net /I2S_LRCLK: track 0.00 -> 41.0 mm, vias 0 -> 1
- net /Lin: track 0.00 -> 40.5 mm
- net /direction: track 0.00 -> 35.7 mm, vias 0 -> 1
- net /I2S_BCLK: track 0.00 -> 26.7 mm, vias 0 -> 1
- net Net-(J1-Pad1): track 0.00 -> 25.1 mm, vias 0 -> 1
- net GNDA: track 0.00 -> 22.5 mm, vias 0 -> 39
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- added copper zone on B.Cu, net GND
- added copper zone on F.Cu, net GND
- added copper zone on B.Cu, net GNDA
- added copper zone on F.Cu, net GNDA
Other:
- board size 65 x 56 mm -> 65.1 x 65.5 mm
- net class Default: clearance 0.2 -> 0.15; trace_width 0.2 -> 0.15; via_dia 0.9 -> 0.7; via_drill 0.6 -> 0.4
- rule trace_clearance: 0.2 -> 0.15
- rule trace_min: 0.1524 -> 0.15
- rule via_min_drill: 0.5 -> 0.4
- rule via_min_size: 0.8 -> 0.7
- board text added: "Flatmax (C) 2021 RAM Platter Hybrid V1.0"
- board text added: "audioinjector.net"
