File: electronics/RAMPlatterHybrid.kicad_pcb (KiCad board)
At the start: 2 copper layers, 65.1 x 65.5 mm, 48 parts, among them J1 Raspberry_Pi_2_3, J2 Raspberry_Pi_2_3, U1 LM358, U2 74LVC74APW, U3 AV2-8.4-10, U4 AV2-8.4-10, U5 HC4046A, U6 CD74HC4059, U7 AP1117-33, U8 WM8750

Commit message: v1.1 Many hardware bug fixes, 4059 now dividing correctly. 4046 voc on better target, still debugging 4046 PLL.
Parts:
- added JP4: Jumper_2_Open, Jumper:SolderJumper-2_P1.3mm_Open_Pad1.0x1.5mm, B.Cu at (240.1, 118.2)
- added JP5: Jumper_2_Open, Jumper:SolderJumper-2_P1.3mm_Open_Pad1.0x1.5mm, B.Cu at (239.8, 115.8)
- C23: value 20n -> 1n
- R12: value 150k -> 3k
Connections:
- R11 pad 1: Net-(R11-Pad1) -> Net-(JP4-Pad2)
- U5 pad 13: (no net) -> Net-(JP4-Pad1)
- U5 pad 15: (no net) -> Net-(JP5-Pad1)
- U5 pad 2: Net-(R11-Pad1) -> (no net)
- U5 pad 5: +3V3 -> GND
- U6 pad 15: /HIGH -> /LOW
- U6 pad 18: /HIGH -> /LOW
- U6 pad 19: /HIGH -> /LOW
- U6 pad 22: /HIGH -> /LOW
- U6 pad 5: /HIGH -> /LOW
- U6 pad 7: /HIGH -> /LOW
- U6 pad 9: /LOW -> /HIGH
Routing:
- net /HIGH: track 54.9 -> 33.4 mm, vias 11 -> 6
- net Net-(R11-Pad1): track 13.7 -> 0.00 mm, vias 2 -> 0
- net /LOW: track 52.9 -> 64.9 mm, vias 11 -> 12
- net +3V3: track 128.5 -> 117.9 mm, vias 6 -> 5
- net Net-(JP4-Pad2): track 0.00 -> 9.78 mm, vias 0 -> 1
- net Net-(JP5-Pad1): track 0.00 -> 0.30 mm, vias 0 -> 1
- net Net-(JP4-Pad1): track 0.00 -> 0.10 mm, vias 0 -> 1
- net GND: vias 87 -> 86
Other:
- board text added: "Flatmax (C) 2021 RAM Platter Hybrid V1.1"
- board text removed: "Flatmax (C) 2021 RAM Platter Hybrid V1.0"
